File: MEMLNaut_0_2/MEMLNaut_0_2.kicad_pcb (KiCad board)
At the start: 4 copper layers, 155 x 103 mm, 114 parts, among them CN1 MIDI In, CN2 MIDI Out, J1 Hanbo_USB_C_Receptacle_USB2.0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, J10 Line In R, J11 Line In L, J12 SPI1 header, J13 Micro_SD_Card_Det_Hirose_DM3AT, J14 Conn_I2C, J15 Line In Cx, J17 Headphone Cx, J18 Line Out R, J19 Line Out L, J2 Custom Cx, J20 Line Out Cx, J21 Conn_Power_Ext, J3 ADC Cx, J4 GPIO B Cx, J5 GPIO A Cx, J6 Joystick Cx, J7 Conn_Power, J8 Conn_Pi_SWD, J9 mic, SW1 SW on-on toggle, SW2 SW on-on toggle, SW3 SW Momentary (on)-off-(on) 1M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, SW4 SW Momentary (on)-off-(on) 1M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, U1 W25Q128JVPIQ, U10 LP5907MFX-1.8, U2 FLASH or PSRAM, U4 TLV76733DRVR, U5 RP235x-B, U6 TLV76733DRVR, U7 6N138, U8 SGTL5000XNLA3, U9 TFT_320x240, Y1 CM4012M00012001

Commit message: v0.3a
Parts:
- added J22: I2S Cx, emutelab:HDR-SMD_6P-P2.54-V-M-S4.8, F.Cu at (125.5, 57.2)
- added R22: 0R0, Resistor_SMD:R_0603_1608Metric, F.Cu at (165.4, 59.6)
- added R23: 0R0, Resistor_SMD:R_0603_1608Metric, F.Cu at (166.5, 57.3)
- added R24: 0R0, Resistor_SMD:R_0603_1608Metric, F.Cu at (161.1, 53.6)
- added R25: 0R0, Resistor_SMD:R_0603_1608Metric, F.Cu at (164.6, 54.3)
- added R26: 0R0, Resistor_SMD:R_0603_1608Metric, F.Cu at (166.8, 54.3)
- D2: footprint LED_SMD:LED_0603_1608Metric -> LED_SMD:LED_0805_2012Metric
- J17: value Headphone Cx -> Headphone_Cx
- moved C25 2.62 mm to (161.7, 49.3)
- moved R14 1.66 mm to (160.5, 47.5)
Connections:
- C25 pad 2: /CODEC_GND -> GNDA
- CN1 pad 2: unconnected-(CN1-Pad2) -> Net-(D1-A)
- CN1 pad 5: Net-(D1-A) -> unconnected-(CN1-Pad5)
- CN2 pad 2: GND -> Net-(CN2-Pad2)
- CN2 pad 3: unconnected-(CN2-Pad3) -> GND
- CN2 pad 5: Net-(CN2-Pad5) -> unconnected-(CN2-Pad5)
- R12 pad 1: Net-(CN2-Pad5) -> Net-(CN2-Pad2)
- R15 pad 1: /GPIO10_I2S_MCLK -> Net-(R15-Pad1)
- U8 pad 14: /GPIO9_I2S_LRCLK -> Net-(U8-I2S_LRCLK)
- U8 pad 15: /GPIO8_I2S_BLCK -> Net-(U8-I2S_SCLK)
- U8 pad 16: /GPIO7_I2S_DOUT -> Net-(U8-I2S_DOUT)
- U8 pad 17: /GPIO6_I2S_DIN -> Net-(U8-I2S_DIN)
Routing:
- net /GPIO10_I2S_MCLK: track 105.5 -> 144.6 mm, vias 4 -> 5
- net /GPIO8_I2S_BLCK: track 84.1 -> 123.1 mm, vias 4 -> 5
- net /GPIO6_I2S_DIN: track 70.6 -> 105.3 mm, vias 3 -> 4
- net /GPIO7_I2S_DOUT: track 70.7 -> 104.2 mm, vias 3 -> 4
- net /GPIO9_I2S_LRCLK: track 66.5 -> 99.3 mm, vias 3 -> 4
- net Net-(CN2-Pad2): track 0.00 -> 24.0 mm
- net Net-(D1-A): track 121.2 -> 103.6 mm
- net GNDA: track 303.7 -> 318.9 mm, vias 5 -> 7
- net Net-(U8-I2S_DIN): track 0.00 -> 14.2 mm
- net Net-(CN2-Pad5): track 12.5 -> 0.00 mm
- net Net-(U8-I2S_DOUT): track 0.00 -> 10.6 mm
- net Net-(U8-I2S_LRCLK): track 0.00 -> 10.6 mm
- net Net-(R15-Pad1): track 0.00 -> 5.08 mm
- net Net-(U8-I2S_SCLK): track 0.00 -> 4.28 mm
- net /GPIO13_SPI1_CS: track 161.4 -> 163.4 mm
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Other:
- board text added: "3V3"
- board text added: "3V3Sig"
- board text added: "5V"
- board text added: "5V In"
- board text added: "< GND >"
- board text added: "Bootsel"
- board text added: "Ext Power"
- board text added: "GND"
- board text added: "Headphone"
- board text added: "I2C"
- board text added: "Joystick"
- board text added: "Line In"
- board text added: "Line Out"
- board text added: "MEMLNaut 0.2 Musically Embodied Machine Learning Emute Lab @ University of Sussex April 2025 https://github.com/MusicallyEmbodiedML"
- board text added: "MIDI In"
- board text added: "MIDI Out"
- board text added: "PSRAM"
- board text added: "Reset"
- board text added: "SCL"
- board text added: "SDA"
- board text added: "SWD"
- board text added: "mic"
- board text added: "power"
- board text removed: "MEMLNaut 0.1 Musically Embodied Machine Learning University of Sussex March 2025 https://github.com/MusicallyEmbodiedML"
