File: MEMLNaut_0_2/MEMLNaut_0_2.kicad_sch (KiCad schematic)
At the start: 109 parts, among them CN1 MIDI In, CN2 MIDI Out, J1 Hanbo_USB_C_Receptacle_USB2.0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, J10 Line In R, J11 Line In L, J12 SPI1 header, J13 Micro_SD_Card_Det_Hirose_DM3AT, J14 Conn_I2C, J15 Line In Cx, J17 Headphone Cx, J18 Line Out R, J19 Line Out L, J2 Custom Cx, J20 Line Out Cx, J21 Conn_Power_Ext, J3 ADC Cx, J4 GPIO B Cx, J5 GPIO A Cx, J6 Joystick Cx, J7 Conn_Power, J8 Conn_Pi_SWD, J9 mic, SW1 SW on-on toggle, SW2 SW on-on toggle, SW3 SW Momentary (on)-off-(on) 1M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, SW4 SW Momentary (on)-off-(on) 1M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, U1 W25Q128JVPIQ, U10 LP5907MFX-1.8, U2 FLASH or PSRAM, U4 TLV76733DRVR, U5 RP235x-B, U6 TLV76733DRVR, U7 6N138, U8 SGTL5000XNLA3, U9 TFT_320x240, Y1 CM4012M00012001

Commit message: v0.3a
Parts:
- added J22: I2S Cx, emutelab:HDR-SMD_6P-P2.54-V-M-S4.8, symbol Connector_Generic:Conn_01x06
- added R22, R23, R24, R25, R26: 0R0, Resistor_SMD:R_0603_1608Metric, symbol Device:R
- D2: footprint LED_SMD:LED_0603_1608Metric -> LED_SMD:LED_0805_2012Metric
- J17: value Headphone Cx -> Headphone_Cx
Connections:
- net CODEC_GND is gone; now on net GNDA: C25.2
- net GND: now also CN2.3, J22.1 (Pin_1); no longer CN2.2
- net GPIO10_I2S_MCLK: now also J22.2 (Pin_2), R22.1; no longer R15.1
- net GPIO6_I2S_DIN: now also J22.6 (Pin_6), R26.1; no longer U8.17 (I2S_DIN)
- net GPIO7_I2S_DOUT: now also J22.5 (Pin_5), R25.1; no longer U8.16 (I2S_DOUT)
- net GPIO8_I2S_BLCK: now also J22.4 (Pin_4), R24.1; no longer U8.15 (I2S_SCLK)
- net GPIO9_I2S_LRCLK: now also J22.3 (Pin_3), R23.1; no longer U8.14 (I2S_LRCLK)
- net at D1.2 (A), U7.3 (C2): now also CN1.2; no longer CN1.5
- net at R12.1: now also CN2.2; no longer CN2.5
- new net: R25.2, U8.16 (I2S_DOUT)
- new net: R15.1, R22.2
- new net: R26.2, U8.17 (I2S_DIN)
- new net: R23.2, U8.14 (I2S_LRCLK)
- new net: R24.2, U8.15 (I2S_SCLK)
- no-connect marks 25 -> 24
Other:
- moved on the sheet: R11, R12
